Commit message: fix(p7): correct URDF joint axis directions and J2 limits after real-arm sign-check (#156)
Closes #154

实机正方向核对(sign-check)后修正 P7 URDF 的关节轴向与 J2 限位。

## 变更
- `p7__left.urdf` / `p7__right.urdf`：翻转相关关节 `axis` 方向；对调 J2 `limit` 上下限（lower/upper）

Reviewed-on: https://gitea.linkerhub.work/linker-bot/linkerbot-python-sdk/pulls/156
Co-authored-by: sunyutong <yutong.sun25@gmail.com>
Co-committed-by: sunyutong <yutong.sun25@gmail.com>

File: src/linkerbot/arm/kinetix/urdf/p7__left.urdf (robot description, URDF)
Before this commit: robot lkls73_arm_left, 9 links, 8 joints
Joints:
- joint L1_Joint: axis 0 -1 0 -> 0 1 0
- joint L2_Joint: axis -1 0 0 -> 1 0 0; limit lower=-3.2 upper=0.07 effort=80 velocity=10.47 -> lower=-0.07 upper=3.2 effort=80 velocity=10.47
- joint L3_Joint: axis 0 0 1 -> 0 0 -1
- joint L4_Joint: axis 0 -1 0 -> 0 1 0
- joint L5_Joint: axis 0 0 1 -> 0 0 -1
- joint L6_Joint: axis 0 -1 0 -> 0 1 0
- joint L7_Joint: axis -1 0 0 -> 1 0 0

File: src/linkerbot/arm/kinetix/urdf/p7__right.urdf (robot description, URDF)
Before this commit: robot lkls73_arm_right, 9 links, 8 joints
Joints:
- joint R1_Joint: axis 0 1 0 -> 0 -1 0
- joint R2_Joint: axis -1 0 0 -> 1 0 0; limit lower=-0.07 upper=3.2 effort=80 velocity=10.47 -> lower=-3.2 upper=0.07 effort=80 velocity=10.47
- joint R3_Joint: axis 0 0 1 -> 0 0 -1
- joint R5_Joint: axis 0 0 1 -> 0 0 -1
- joint R7_Joint: axis -1 0 0 -> 1 0 0
